Commit message: update new lidar working (proper mapping still out for testing)

File: src/eagle_bot/description/lidar.xacro (robot description, xacro)
@@ -4,5 +4,5 @@
         <parent link="chassis"/>
         <child link="laser_frame"/>
-        <origin xyz="0.43 0 0.330" rpy="0 0 0"/>
+        <origin xyz="0.405 0 0.260" rpy="0 0 0"/>
     </joint>
     <link name="laser_frame">

Commit message: changed lidarn position

File: src/eagle_bot/description/lidar.xacro (robot description, xacro)
@@ -4,5 +4,5 @@
         <parent link="chassis"/>
         <child link="laser_frame"/>
-        <origin xyz="0.405 0 0.260" rpy="0 0 0"/>
+        <origin xyz="0.405 0 0.260" rpy="0 0 3.14"/>
     </joint>
     <link name="laser_frame">

Commit message: Added LiDAR 180 degree rotation fix

File: src/eagle_bot/description/lidar.xacro (robot description, xacro)
@@ -19,5 +19,5 @@
         </collision>
         <xacro:inertial_cylinder mass="0.1" length="0.04" radius="0.05">
-            <origin xyz="0 0 0" rpy="0 0 0"/>
+            <origin xyz="0 0 0" rpy="0 0 3.14159265359"/>
         </xacro:inertial_cylinder>
     </link>
